File: Kicad/Cellox/XLR_input.sch (KiCad schematic (older format))
At the start: 0 parts

Commit message: Add input stage + clipping stage
Parts:
- added C? (x5): 47µ, symbol Device:C
- added C? (x2): 2µ, symbol Device:C
- added Q?: MMBT2222A, symbol Device:Q_NPN_BEC
- added R? (x2): 100k, symbol Device:R
- added R?: 100, symbol Device:R
- added R?: 48k, symbol Device:R
- added R?: 10k, symbol Device:R
- added R?: 4,8k, symbol Device:R
- added R? (x2): 480, symbol Device:R
- added U?: INA597, symbol schematic_symbols_cellox:INA597
Connections:
- new net: C?.1, R?.1, R?.1, R?.2
- new net: C?.1, U?.5 (Sense)
- new net: C?.2, U?.1 (REF)
- new net: C?.2, U?.2 (-IN), U?.6 (Out)
- new net: C?.1, Q?.1 (B), R?.1, R?.2
- new net: C?.2, Q?.3 (C), R?.2
- new net: C?.1, C?.1, R?.1, R?.2
- new net: Q?.2 (E), R?.1
- new net +48V: R?.1
- new net +9V: R?.1, R?.1, U?.7 (V+)
- new net GND: C?.2, C?.2, C?.2, R?.2, R?.2, U?.4 (V-)
- new net Signal+: C?.2, R?.2
- new net Signal-: C?.1, R?.2
- new net SignalOut: C?.1
- new net Vref: U?.3 (+IN)
