File: Kicad/Cellox/Distortion_Tone_Volume.sch (KiCad schematic (older format))
At the start: 13 parts

Commit message: Commit, I forget
Parts:
- removed C?: C, symbol Device:C
- removed D? (x2): D, symbol Device:D
- added C? (x2): 220n, symbol Device:C
- added C? (x2): C, symbol Device:C
- added C?: 10µ, symbol Device:C
- added D? (x2): D, symbol Device:D
- added D? (x2): LED, symbol Device:LED
- added Q? (x2): MMBFJ201, symbol Device:Q_NJFET_DGS
- added R?: 220, symbol Device:R
- added RV?: 20k lin, symbol Device:R_POT
- added RV?: 500k log, symbol Device:R_POT
- added SW?: SK14D01G6, symbol schematic_symbols_cellox:SK14D01G6
- C?: value C -> 20µ
- R?: value R -> 51k
- R?: value R -> 100k
- RV?: value R_POT -> 500k lin
Connections:
- net labels added: +9V, SW_S_In, SW_S_Out
- wire segments 34 -> 93
- no-connect marks 1 -> 2
Other:
- moved on the sheet: U?C
