File: Kicad/Cellox/Simulations/Simulation_XLR_Input.sch (KiCad schematic (older format))
At the start: 8 parts, among them Q1 2N3904

Commit message: Commit, I forget
Parts:
- removed Q1: 2N3904, Package_TO_SOT_THT:TO-92_Inline, symbol Transistor_BJT:2N3904
- removed R7: 3.3k, symbol Device:R
- C1: value 1000000u -> 10u
- R1, R2: value 20k -> 18k
- V1: Spice_Model dc 0 ac 1 sin(0 5 1k) -> dc 0 ac 1 sin(0 1 1k)
- V2: value dc 15 ac 0 -> dc 9 ac 0
Changed lines of the file:
@@
 P 4800 4700
 F 0 "V2" H 5028 4746 50  0000 L CNN
-F 1 "dc 15 ac 0" H 5028 4655 50  0000 L CNN
+F 1 "dc 9 ac 0" H 5028 4655 50  0000 L CNN
 F 2 "" H 4800 4700 50  0001 C CNN
 F 3 "~" H 4800 4700 50  0001 C CNN
@@
 F 3 "~" H 8350 3150 50  0001 C CNN
 F 4 "V" H 8350 3150 50  0001 C CNN "Spice_Primitive"
-F 5 "dc 0 ac 1 sin(0 5 1k)" H 8350 3150 50  0001 C CNN "Spice_Model"
+F 5 "dc 0 ac 1 sin(0 1 1k)" H 8350 3150 50  0001 C CNN "Spice_Model"
 F 6 "Y" H 8350 3150 50  0001 C CNN "Spice_Netlist_Enabled"
 	1    8350 3150
@@
 P 9200 3500
 F 0 "R2" H 9270 3546 50  0000 L CNN
-F 1 "20k" H 9270 3455 50  0000 L CNN
+F 1 "18k" H 9270 3455 50  0000 L CNN
 F 2 "" V 9130 3500 50  0001 C CNN
 F 3 "~" H 9200 3500 50  0001 C CNN
 	1    9200 3500
-	1    0    0    -1
-$EndComp
-$Comp
-L Device:R R7
-U 1 1 60B34009
-P 10050 3450
-F 0 "R7" H 10120 3496 50  0000 L CNN
-F 1 "3.3k" H 10120 3405 50  0000 L CNN
-F 2 "" V 9980 3450 50  0001 C CNN
-F 3 "~" H 10050 3450 50  0001 C CNN
-	1    10050 3450
-	1    0    0    -1
-$EndComp
-$Comp
-L power:GND #PWR04
-U 1 1 60B37061
-P 10050 3650
-F 0 "#PWR04" H 10050 3400 50  0001 C CNN
-F 1 "GND" H 10055 3477 50  0000 C CNN
-F 2 "" H 10050 3650 50  0001 C CNN
-F 3 "" H 10050 3650 50  0001 C CNN
-	1    10050 3650
 	1    0    0    -1
 $EndComp
@@
 Wire Wire Line
 	9200 3650 9200 4050
-Wire Wire Line
-	10050 3300 10050 3200
-Wire Wire Line
-	9750 3000 9250 3000
 Connection ~ 9250 3000
 Wire Wire Line
 	9250 3000 9250 3350
-Text Label 10050 3250 0    50   ~ 0
-Vout
 $Comp
 L power:GND #PWR0103
@@
 P 8850 3000
 F 0 "C1" V 9102 3000 50  0000 C CNN
-F 1 "1000000u" V 9011 3000 50  0000 C CNN
+F 1 "10u" V 9011 3000 50  0000 C CNN
 F 2 "" H 8888 2850 50  0001 C CNN
 F 3 "~" H 8850 3000 50  0001 C CNN
@@
 	8350 3450 8350 3700
 $Comp
-L power:+9V #PWR0106
-U 1 1 60B4BEB2
-P 10000 2650
-F 0 "#PWR0106" H 10000 2500 50  0001 C CNN
-F 1 "+9V" H 10000 2800 50  0000 C CNN
-F 2 "" H 10000 2650 50  0001 C CNN
-F 3 "" H 10000 2650 50  0001 C CNN
-	1    10000 2650
-	1    0    0    -1
-$EndComp
-Wire Wire Line
-	10000 2650 10050 2650
-Wire Wire Line
-	10050 2650 10050 2800
-Wire Wire Line
-	10050 3600 10050 3650
-$Comp
 L Device:R R1
 U 1 1 60B4F88A
 P 9250 2650
 F 0 "R1" H 9320 2696 50  0000 L CNN
-F 1 "20k" H 9320 2605 50  0000 L CNN
+F 1 "18k" H 9320 2605 50  0000 L CNN
 F 2 "" V 9180 2650 50  0001 C CNN
 F 3 "~" H 9250 2650 50  0001 C CNN
@@
 	1    0    0    -1
 $EndComp
-$Comp
-L Transistor_BJT:2N3904 Q1
-U 1 1 60B50A5B
-P 9950 3000
-F 0 "Q1" H 10140 3046 50  0000 L CNN
-F 1 "2N3904" H 10140 2955 50  0000 L CNN
-F 2 "Package_TO_SOT_THT:TO-92_Inline" H 10150 2925 50  0001 L CIN
-F 3 "https://www.fairchildsemi.com/datasheets/2N/2N3904.pdf" H 9950 3000 50  0001 L CNN
-F 4 "Q" H 9950 3000 50  0001 C CNN "Spice_Primitive"
-F 5 "DI_MMBT2222A" H 9950 3000 50  0001 C CNN "Spice_Model"
-F 6 "Y" H 9950 3000 50  0001 C CNN "Spice_Netlist_Enabled"
-F 7 "PspiceModel\\MMBT2222A\\MMBT2222A.lib" H 9950 3000 50  0001 C CNN "Spice_Lib_File"
-	1    9950 3000
-	1    0    0    -1
-$EndComp
